Commit message: updated proximty calculations, creating scenes, visualizations

File: data_collection/object_sets/setup/box.urdf (robot description, URDF)
Before this commit: robot cube.urdf, 1 links, 0 joints
Links:
- link base_link: geometry collision mesh filename=box.obj scale=0.0125 0.005 0.0125; visual mesh filename=box.obj scale=0.0125 0.005 0.0125
